File: Safe&Sound KiCad Project/Safe&Sound PCB.kicad_sch (KiCad schematic)
At the start: 36 parts, among them J2 Conn_01x02_Female, J4 Conn_01x03_Female, J5 Conn_01x05_Female, J6 Conn_01x07_Female, SW1 EN, SW2 BT, SW3 BOOT, U1 ESP32-WROOM-32, U2 MCP1825T-3302E/DC

Commit message: huella switch
Parts:
- C1: value (none) -> 100n; footprint (none) -> Capacitor_SMD:C_0805_2012Metric_Pad1.18x1.45mm_HandSolder
- C2, C3, C4, C5, C6, C7, C8: footprint (none) -> Capacitor_SMD:C_0805_2012Metric_Pad1.18x1.45mm_HandSolder
- D1: footprint (none) -> LED_SMD:LED_0805_2012Metric_Pad1.15x1.40mm_HandSolder
- J1: value (none) -> USB_B_Micro; footprint (none) -> Connector_USB:USB_Micro-B_Molex-105017-0001
- J3: value (none) -> Conn_01x03_Female; footprint (none) -> Connector_PinSocket_2.54mm:PinSocket_1x03_P2.54mm_Vertical
- R1, R10, R11, R2, R3, R4, R5, R6, R7, R8, R9: footprint (none) -> Resistor_SMD:R_0805_2012Metric_Pad1.20x1.40mm_HandSolder
- RV1: value (none) -> R_Potentiometer; footprint (none) -> Potentiometer_SMD:Potentiometer_ACP_CA6-VSMD_Vertical
- SW1, SW2, SW3: footprint (none) -> Button_Switch_SMD:SW_SPST_EVQQ2
- SW4: value (none) -> BT; footprint (none) -> Button_Switch_SMD:SW_SPST_EVQQ2
- SW5: value (none) -> SW_SPDT; footprint (none) -> Button_Switch_SMD:SW_DPDT_CK_JS202011JCQN
- U2: footprint (none) -> MCP1825T-3302E_DC:SOT230P700X180-6N
- U3: value (none) -> MCP73831-2-OT; footprint (none) -> Package_TO_SOT_SMD:SOT-23-5_HandSoldering
